Commit message: wheel control added

File: snakewbot_description/urdf/snake.urdf.xacro (robot description, xacro)
@@ -7,5 +7,5 @@
   <!-- BASE-FOOTPRINT -->
   <!-- base_footprint is a fictitious link(frame) that is on the ground right below base_link origin -->
-	<link name="base_footprint1.0">
+	<link name="base_footprint1">
 		<inertial>
             <mass value="0.0001" />
@@ -26,13 +26,32 @@
         </visual>
     </link>
-    <snake_module number="1.0" rotY="0" rotZ="0"/>
-    <snake_module number="2.0" rotY="0" rotZ="0"/>
+    <snake_module number="1" n2="2" rotY="0" rotZ="0"/>
+    <snake_module number="2" n2="3" rotY="0" rotZ="0"/>
+    <snake_module number="3" n2="4" rotY="0" rotZ="0"/>
+    <snake_module number="4" n2="5" rotY="0" rotZ="0"/>
+    <snake_module number="5" n2="6" rotY="0" rotZ="0"/>
+    <snake_module number="6" n2="7" rotY="0" rotZ="0"/>
+    <snake_module number="7" n2="8" rotY="0" rotZ="0"/>
+    <snake_module number="8" n2="9" rotY="0" rotZ="0"/>
+  <gazebo>
+    <plugin name="skid_steer_drive_controller8" filename="libgazebo_ros_skid_steer_drive.so">
+      <alwaysOn>true</alwaysOn>
+      <updateRate>100.0</updateRate>
+      <leftFrontJoint>front_left8_wheel_joint</leftFrontJoint>
+      <rightFrontJoint>front_right8_wheel_joint</rightFrontJoint>
+      <leftRearJoint>back_left8_wheel_joint</leftRearJoint>
+      <rightRearJoint>back_right8_wheel_joint</rightRearJoint>
+      <wheelSeparation>${base_y_size}</wheelSeparation>
+      <wheelDiameter>${2*wheel_radius}</wheelDiameter>
+      <torque>35</torque>
+      <broadcastTF>1</broadcastTF>
+      <odometryFrame>map</odometryFrame>
+      <commandTopic>cmd_vel</commandTopic>
+      <odometryTopic>odom</odometryTopic>
+      <robotBaseFrame>base_footprint8</robotBaseFrame>
+    </plugin>
 <!--
-    <snake_module number="3.0" rotY="0" rotZ="0"/>
-    <snake_module number="4.0" rotY="0" rotZ="0"/>
-    <snake_module number="5.0" rotY="0" rotZ="0"/>
-    <snake_module number="6.0" rotY="0" rotZ="0"/>
-    <snake_module number="7.0" rotY="0" rotZ="0"/>
-    <snake_module number="8.0" rotY="0" rotZ="0"/>
+    <plugin name="gazebo_ros_control" filename="libgazebo_ros_control.so" />
 -->
+  </gazebo>
 </robot>

File: snakewbot_description/urdf/snake_module.urdf.xacro (robot description, xacro)
@@ -16,5 +16,5 @@
               izz="${m*(x*x+z*z)/12}" />
   </macro>
-  <xacro:macro name="snake_module" params="number rotY rotZ">
+  <xacro:macro name="snake_module" params="number n2 rotY rotZ">
 	<joint name="base_footprint_joint${number}" type="fixed">
 		<origin xyz="0 0 ${wheel_radius - base_z_origin_to_wheel_origin}" rpy="0 0 0" />
@@ -125,7 +125,7 @@
 		<origin xyz="${joint_distance} 0 -${wheel_radius}" rpy="0 0 0" />
 		<parent link="link_z${number}"/>
-		<child link="base_footprint${number+1}" />
+		<child link="base_footprint${n2}" />
 	</joint>
-	<link name="base_footprint${number+1}">
+	<link name="base_footprint${n2}">
 		<inertial>
 			<mass value="0.0001" />

File: snakewbot_description/urdf/wheel.urdf.xacro (robot description, xacro)
@@ -44,8 +44,8 @@
       <turnGravityOff>false</turnGravityOff>
     </gazebo>
+    <joint name="${fb}_${lr}_wheel_joint" type="continuous">
 <!--
-    <joint name="${fb}_${lr}_wheel_joint" type="continuous">
+	<joint name="${fb}_${lr}_wheel_joint" type="fixed">
 -->
-	<joint name="${fb}_${lr}_wheel_joint" type="fixed">
       <parent link="${parent}"/>
       <child link="${fb}_${lr}_wheel"/>
@@ -56,5 +56,4 @@
     </joint>
     <!-- Transmission is important to link the joints and the controller -->
-<!--
     <transmission name="${fb}_${lr}_wheel_joint_trans">
       <type>transmission_interface/SimpleTransmission</type>
@@ -65,5 +64,4 @@
       </actuator>
     </transmission>
--->
   </xacro:macro>
 </robot>

Commit message: wheel control

File: snakewbot_description/urdf/snake.urdf.xacro (robot description, xacro)
@@ -35,23 +35,20 @@
     <snake_module number="8" n2="9" rotY="0" rotZ="0"/>
   <gazebo>
-    <plugin name="skid_steer_drive_controller8" filename="libgazebo_ros_skid_steer_drive.so">
+    <plugin name="skid_steer_drive_controller1" filename="libgazebo_ros_skid_steer_drive.so">
       <alwaysOn>true</alwaysOn>
       <updateRate>100.0</updateRate>
-      <leftFrontJoint>front_left8_wheel_joint</leftFrontJoint>
-      <rightFrontJoint>front_right8_wheel_joint</rightFrontJoint>
-      <leftRearJoint>back_left8_wheel_joint</leftRearJoint>
-      <rightRearJoint>back_right8_wheel_joint</rightRearJoint>
-      <wheelSeparation>${base_y_size}</wheelSeparation>
+      <leftFrontJoint>front_left1_wheel_joint</leftFrontJoint>
+      <rightFrontJoint>front_right1_wheel_joint</rightFrontJoint>
+      <leftRearJoint>back_left1_wheel_joint</leftRearJoint>
+      <rightRearJoint>back_right1_wheel_joint</rightRearJoint>
+      <wheelSeparation>${2*base_y_origin_to_wheel_origin}</wheelSeparation>
       <wheelDiameter>${2*wheel_radius}</wheelDiameter>
       <torque>35</torque>
       <broadcastTF>1</broadcastTF>
       <odometryFrame>map</odometryFrame>
-      <commandTopic>cmd_vel</commandTopic>
+      <commandTopic>/cmd_vel</commandTopic>
       <odometryTopic>odom</odometryTopic>
-      <robotBaseFrame>base_footprint8</robotBaseFrame>
+      <robotBaseFrame>base_footprint1</robotBaseFrame>
     </plugin>
-<!--
-    <plugin name="gazebo_ros_control" filename="libgazebo_ros_control.so" />
--->
   </gazebo>
 </robot>

File: snakewbot_description/urdf/snake_module.urdf.xacro (robot description, xacro)
@@ -144,4 +144,26 @@
 		</visual>
 	</link>
+<!--
+  <transmission name="tran_jointy${number}">
+    <type>transmission_interface/SimpleTransmission</type>
+    <joint name="joint_y${number}"/>
+    <actuator name="motor_joint_y${number}">
+      <hardwareInterface>EffortJointInterface</hardwareInterface>
+      <mechanicalReduction>1</mechanicalReduction>
+    </actuator>
+  </transmission>
+  <transmission name="tran_jointz${number}">
+    <type>transmission_interface/SimpleTransmission</type>
+    <joint name="joint_z${number}"/>
+    <actuator name="motor_joint_z${number}">
+      <hardwareInterface>EffortJointInterface</hardwareInterface>
+      <mechanicalReduction>1</mechanicalReduction>
+    </actuator>
+  </transmission>
+  <gazebo>
+	<plugin name="gazebo_ros_control${number}" filename="libgazebo_ros_control.so" />
+	<robotNamespace>/snakewbot</robotNamespace>
+  </gazebo>
+-->
   </xacro:macro>
 </robot>

File: snakewbot_description/urdf/wheel.urdf.xacro (robot description, xacro)
@@ -26,5 +26,5 @@
         <origin xyz="0 0 0" rpy="${flipY*M_PI/2} 0 0" />
         <geometry>
-          <mesh filename="package://snakewbot_description/meshes/omniwheel.stl" />
+          <cylinder length="${wheel_height}" radius="${wheel_radius}" />
         </geometry>
       </collision>
@@ -45,7 +45,4 @@
     </gazebo>
     <joint name="${fb}_${lr}_wheel_joint" type="continuous">
-<!--
-	<joint name="${fb}_${lr}_wheel_joint" type="fixed">
--->
       <parent link="${parent}"/>
       <child link="${fb}_${lr}_wheel"/>
